File: Dave's KiCad file/IS.sch (KiCad schematic (older format))
At the start: 0 parts

Commit message: IS Work in progress
Done draft L1 diagram in KiCad and some work on the IS L1 docx
Connections:
- net labels added: 0x001, ABUS, ADDR_SEL, AIS_ROM, AIS_Ra#, AIS_Rb#, AIS_TMP2, AS_ALUO, CLOCK, DATA_SEL, DBUS, FLAGS, ID_TMP1, ID_TMP2, IS_0x1, IS_ROM, IS_TMP1, IS_TMP2, JBITS, MODE, OLS, OPCODE, READ, RESET, Ra#, Rb#, SD_AA, SD_AB, SD_PC, SD_PN, SD_PV, SD_RD, SEQ#, SEQ_ADDR, SEQ_END, SS_AO, SS_PC, SS_PV, SS_RD, WRITE
- wire segments 0 -> 59
Other:
- note added: "16 BIT \nTRISTATE\n BUFFER"
- note added: "CLOCK\nGENERATOR"
- note added: "INPUTS"
- note added: "OPCODE\n LATCH"
- note added: "OUTPUTS"
- note added: "POWER UP\n RESET"
- note added: "RAM ADDRESS\n CONTROL"
- note added: "SEQUENCE\n CONTROL"
- note added: "SEQUENCE\n ROM"
- note added: "TEMP 16 BIT\n LATCH1"
- note added: "TEMP 16 BIT\n LATCH2"
