File: Dave's KiCad file/L2SeqCtrl.sch (KiCad schematic (older format))
At the start: 0 parts

Commit message: Work in progress
Connections:
- wire segments 19 -> 27
Other:
- note added: "5 BIT \nCOUNTER"
Changed lines of the file:
@@
 $Descr A4 11693 8268
 encoding utf-8
-Sheet 2 2
+Sheet 1 1
 Title ""
 Date ""
@@
 Comment4 ""
 $EndDescr
-Text Label 3400 3900 0    50   ~ 0
+Text Label 3150 3900 0    50   ~ 0
 JBITS
 Wire Notes Line
-	3350 3600 3750 3600
-Text Notes 3400 3600 0    50   ~ 0
+	3100 3400 3500 3400
+Text Notes 3150 3400 0    50   ~ 0
 INPUTS
-Text Notes 7000 3750 0    50   ~ 0
+Text Notes 5600 3700 0    50   ~ 0
 OUTPUTS
-Text Label 3400 3700 0    50   ~ 0
+Text Label 3150 3700 0    50   ~ 0
 SEQ_END
-Wire Wire Line
-	3400 3700 3750 3700
-Text Label 3400 3800 0    50   ~ 0
+Text Label 3150 3800 0    50   ~ 0
 FLAGS
-Text Label 3400 4000 0    50   ~ 0
+Text Label 3150 4000 0    50   ~ 0
 SEQ#
-Wire Wire Line
-	3400 4100 3750 4100
-Text Label 3400 4100 0    50   ~ 0
+Text Label 3150 3500 0    50   ~ 0
 CLOCK
-Wire Wire Line
-	3750 4200 3400 4200
-Text Label 3400 4200 0    50   ~ 0
+Text Label 3150 3600 0    50   ~ 0
 RESET
 Wire Notes Line
-	3750 4250 3350 4250
-Wire Notes Line
-	3750 3600 3750 4250
-Wire Notes Line
-	3350 3600 3350 4250
-Text Label 7350 3850 2    50   ~ 0
+	3500 4050 3100 4050
+Wire Notes Line
+	3500 3400 3500 4050
+Wire Notes Line
+	3100 3400 3100 4050
+Text Label 5950 3900 2    50   ~ 0
 SEQ_ADDR
-Text Label 7350 3950 2    50   ~ 0
+Text Label 5950 3800 2    50   ~ 0
 OLS
-Wire Wire Line
-	7350 3950 6950 3950
-Wire Notes Line
-	7400 3750 7400 4000
-Wire Bus Line
-	6750 3850 7350 3850
-Entry Wire Line
-	6650 3500 6750 3600
-Entry Wire Line
-	6650 3600 6750 3700
-Entry Wire Line
-	6650 3700 6750 3800
-Entry Wire Line
-	6650 3800 6750 3900
-Entry Wire Line
-	6650 3900 6750 4000
-Entry Wire Line
-	6650 4000 6750 4100
-Entry Wire Line
-	6650 4100 6750 4200
-Entry Wire Line
-	6650 4200 6750 4300
-Entry Wire Line
-	6650 4300 6750 4400
-Entry Wire Line
-	6650 3400 6750 3500
-Wire Wire Line
-	6650 4300 6550 4300
-Text Label 6550 4300 0    50   ~ 0
+Wire Notes Line
+	6000 3700 6000 3950
+Entry Wire Line
+	5250 3450 5350 3550
+Entry Wire Line
+	5250 3550 5350 3650
+Entry Wire Line
+	5250 3650 5350 3750
+Entry Wire Line
+	5250 3750 5350 3850
+Entry Wire Line
+	5250 3900 5350 4000
+Entry Wire Line
+	5250 4000 5350 4100
+Entry Wire Line
+	5250 4100 5350 4200
+Entry Wire Line
+	5250 4200 5350 4300
+Entry Wire Line
+	5250 4300 5350 4400
+Entry Wire Line
+	5250 3350 5350 3450
+Wire Wire Line
+	5250 4300 5150 4300
+Text Label 5150 4300 0    50   ~ 0
 A9
 Wire Wire Line
-	6650 3400 6550 3400
-Wire Wire Line
-	6650 3500 6550 3500
-Wire Wire Line
-	6650 3600 6550 3600
-Wire Wire Line
-	6650 3700 6550 3700
-Wire Wire Line
-	6650 3800 6550 3800
-Wire Wire Line
-	6650 3900 6550 3900
-Wire Wire Line
-	6650 4000 6550 4000
-Wire Wire Line
-	6650 4100 6550 4100
-Wire Wire Line
-	6650 4200 6550 4200
-Text Label 6550 4200 0    50   ~ 0
+	5250 3350 5150 3350
+Wire Wire Line
+	5250 3450 5150 3450
+Wire Wire Line
+	5250 3550 5150 3550
+Wire Wire Line
+	5250 3650 5150 3650
+Wire Wire Line
+	5250 3750 5150 3750
+Wire Wire Line
+	5250 3900 5150 3900
+Wire Wire Line
+	5250 4000 5150 4000
+Wire Wire Line
+	5250 4100 5150 4100
+Wire Wire Line
+	5250 4200 5150 4200
+Text Label 5150 4200 0    50   ~ 0
 A8
-Text Label 6550 4100 0    50   ~ 0
+Text Label 5150 4100 0    50   ~ 0
 A7
-Text Label 6550 4000 0    50   ~ 0
+Text Label 5150 4000 0    50   ~ 0
 A6
-Text Label 6550 3900 0    50   ~ 0
+Text Label 5150 3900 0    50   ~ 0
 A5
-Text Label 6550 3800 0    50   ~ 0
+Text Label 5150 3750 0    50   ~ 0
 A4
-Text Label 6550 3700 0    50   ~ 0
+Text Label 5150 3650 0    50   ~ 0
 A3
-Text Label 6550 3600 0    50   ~ 0
+Text Label 5150 3550 0    50   ~ 0
 A2
-Text Label 6550 3500 0    50   ~ 0
+Text Label 5150 3450 0    50   ~ 0
 A1
-Text Label 6550 3400 0    50   ~ 0
+Text Label 5150 3350 0    50   ~ 0
 A0
 Entry Wire Line
-	6450 4000 6550 3900
-Entry Wire Line
-	6450 4100 6550 4000
-Entry Wire Line
-	6450 4200 6550 4100
-Entry Wire Line
-	6450 4300 6550 4200
-Entry Wire Line
-	6450 4400 6550 4300
-Wire Bus Line
-	6450 3900 6150 3900
-Wire Bus Line
-	6450 4400 6150 4400
-Text Label 6400 4400 2    50   ~ 0
-LSEQ#
-Text Label 6400 3900 2    50   ~ 0
+	5050 4000 5150 3900
+Entry Wire Line
+	5050 4100 5150 4000
+Entry Wire Line
+	5050 4200 5150 4100
+Entry Wire Line
+	5050 4300 5150 4200
+Entry Wire Line
+	5050 4400 5150 4300
+Text Label 4350 3450 0    50   ~ 0
 STEP#
 Entry Wire Line
-	6450 3500 6550 3400
-Entry Wire Line
-	6450 3600 6550 3500
-Entry Wire Line
-	6450 3700 6550 3600
-Entry Wire Line
-	6450 3800 6550 3700
-Entry Wire Line
-	6450 3900 6550 3800
-Connection ~ 6750 3850
-Wire Notes Line
-	6950 4000 6950 3750
-Wire Notes Line
-	6950 3750 7400 3750
-Wire Notes Line
-	6950 4000 7400 4000
-Wire Bus Line
-	3400 3800 4100 3800
-Wire Bus Line
-	3400 3900 4100 3900
+	5050 3450 5150 3350
+Entry Wire Line
+	5050 3550 5150 3450
+Entry Wire Line
+	5050 3650 5150 3550
+Entry Wire Line
+	5050 3750 5150 3650
+Entry Wire Line
+	5050 3850 5150 3750
+Wire Notes Line
+	5550 3950 5550 3700
+Wire Notes Line
+	5550 3700 6000 3700
+Wire Notes Line
+	5550 3950 6000 3950
+Wire Bus Line
+	3150 3800 4100 3800
+Wire Bus Line
+	3150 3900 4100 3900
 Text Notes 4300 4050 1    50   ~ 0
 FOLLOW\nJUMP?
@@
 	4100 3700 4100 4100
 Wire Bus Line
-	3400 4000 3950 4000
+	3150 4000 3950 4000
 Text Label 4500 3900 0    50   ~ 0
 A5
-Connection ~ 3950 4000
 Wire Bus Line
 	3950 4000 4100 4000
@@
 Wire Wire Line
 	4350 3900 4600 3900
-Wire Bus Line
-	4700 4400 5000 4400
 Text Label 5000 4400 2    50   ~ 0
 LSEQ#
+Text Notes 4300 3600 1    50   ~ 0
+  5 BIT \nCOUNTER
+Text Label 4100 3350 2    50   ~ 0
+CLOCK
+Text Label 4100 3450 2    50   ~ 0
+RESET
+Text Label 4100 3550 2    50   ~ 0
+SEQ_END
+Wire Wire Line
+	3750 3550 4100 3550
+Wire Notes Line style solid rgb(0, 255, 0)
+	4100 3200 4100 3650
+Wire Notes Line style solid rgb(0, 255, 0)
+	4100 3650 4350 3650
+Wire Notes Line style solid rgb(0, 255, 0)
+	4350 3650 4350 3200
+Wire Notes Line style solid rgb(0, 255, 0)
+	4350 3200 4100 3200
+Connection ~ 3950 4000
+Wire Wire Line
+	3750 3550 3750 3700
+Wire Wire Line
+	3150 3700 3750 3700
+Wire Wire Line
+	3650 3450 3650 3600
+Wire Wire Line
+	3150 3600 3650 3600
+Wire Wire Line
+	3650 3450 4100 3450
+Wire Wire Line
+	3550 3350 3550 3500
+Wire Wire Line
+	3150 3500 3550 3500
+Wire Wire Line
+	3550 3350 4100 3350
+Wire Bus Line
+	4700 4400 5050 4400
+Wire Bus Line
+	4350 3450 5050 3450
+Wire Bus Line
+	5350 3900 5950 3900
+Connection ~ 5350 3900
+Wire Wire Line
+	5450 3800 5450 3250
+Wire Wire Line
+	5450 3250 4350 3250
+Wire Wire Line
+	5450 3800 5950 3800
+Wire Bus Line
+	4700 4000 4700 4400
 Wire Bus Line
 	3950 4000 3950 4400
 Wire Bus Line
-	6450 3500 6450 3900
-Wire Bus Line
-	6450 4000 6450 4400
-Wire Bus Line
-	6750 3500 6750 3850
-Wire Bus Line
-	4700 4000 4700 4400
-Wire Bus Line
-	6750 3850 6750 4400
+	5050 3450 5050 3850
+Wire Bus Line
+	5050 4000 5050 4400
+Wire Bus Line
+	5350 3450 5350 3900
+Wire Bus Line
+	5350 3900 5350 4400
+Text Label 4350 3250 0    50   ~ 0
+OLS
 $EndSCHEMATC
